File: kicad_handsolder/MHzDisplayBlaster.kicad_pcb (KiCad board)
At the start: 2 copper layers, 39.6 x 31.2 mm, 5 parts, among them J1 Conn_02x15 DigitRHS, J2 Conn_02x15 DigitLHS, J4 Conn_01x07, U1 DC56-11GWA

Commit message: Update
Parts:
- removed J1: Conn_02x15 DigitRHS, Connector_PinHeader_2.54mm:PinHeader_2x15_P2.54mm_Vertical
- removed J2: Conn_02x15 DigitLHS, Connector_PinHeader_2.54mm:PinHeader_2x15_P2.54mm_Vertical
- moved J4 24.4 mm to (120.3, 48.4)
- moved R1 19.8 mm to (135.6, 48.2), turned to 180 degrees
Connections:
- U1 pad 1: DIG1_E -> unconnected-(U1-DIG1_E-Pad1)
- U1 pad 10: DIG2_B -> 3
- U1 pad 11: DIG2_A -> 1
- U1 pad 12: DIG2_F -> 2
- U1 pad 15: DIG1_B -> 3
- U1 pad 16: DIG1_A -> 2
- U1 pad 17: DIG1_G -> 1
- U1 pad 18: DIG1_F -> 1
- U1 pad 2: DIG1_D -> unconnected-(U1-DIG1_D-Pad2)
- U1 pad 3: DIG1_C -> 3
- U1 pad 4: DP -> 3
- U1 pad 5: DIG2_E -> unconnected-(U1-DIG2_E-Pad5)
- U1 pad 6: DIG2_D -> unconnected-(U1-DIG2_D-Pad6)
- U1 pad 7: DIG2_G -> 2
- U1 pad 8: DIG2_C -> 3
- U1 pad 9: DP -> unconnected-(U1-DP2-Pad9)
Routing:
- net 2: track 90.1 -> 2.54 mm, vias 1 -> 0
- net DP: track 77.4 -> 0.00 mm, vias 3 -> 0
- net 1: track 87.1 -> 31.0 mm, vias 1 -> 0
- net DIG2_G: track 52.5 -> 0.00 mm
- net 3: track 87.6 -> 36.8 mm, vias 6 -> 0
- net DIG1_D: track 36.1 -> 0.00 mm, vias 1 -> 0
- net DIG1_C: track 32.7 -> 0.00 mm, vias 1 -> 0
- net DIG1_A: track 31.2 -> 0.00 mm
- net DIG2_C: track 28.7 -> 0.00 mm
- net DIG1_B: track 28.0 -> 0.00 mm, vias 1 -> 0
- net DIG1_E: track 27.9 -> 0.00 mm
- net DIG2_E: track 27.4 -> 0.00 mm
- net DIG2_D: track 26.0 -> 0.00 mm
- net DIG2_A: track 24.7 -> 0.00 mm, vias 1 -> 0
- net DIG2_F: track 15.7 -> 0.00 mm, vias 1 -> 0
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